File: kicad/logicbuddy.kicad_pcb (KiCad board)
At the start: 2 copper layers, 130 x 100 mm, 33 parts, among them J1 USB_C_2PIN, Q1 NPN, Q2 NPN, Q3 NPN, Q4 NPN, Q5 NPN, Q6 NPN, Q7 NPN, SW1 SW_SPST, SW2 SW_SPST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

Commit message: Reapply "updated labels and fixed footprints"
This reverts commit 2a946a7896d612220efc5a586cb72ca7f3163489.
Parts:
- renumbered R12 to R10, R13 to R11, R3 to R12, R11 to R13, R10 to R3

Commit message: Revert "updated labels and fixed footprints"
This reverts commit cc8675b157493e85bb3edc9923989f4c8e1865eb.
Parts:
- renumbered R3 to R10, R13 to R11, R10 to R12, R11 to R13, R12 to R3
